File: knobber/LED_lighting.kicad_sch (KiCad schematic)
At the start: 34 parts, among them U201 SN74LV1T34DBV

Commit message: updated schematic
Parts:
- C201, C202, C203, C204, C205, C206, C207, C208, C209, C210, C211, C212, C213, C214, C215, C216, C217: footprint Capacitor_SMD:C_0805_2012Metric -> Capacitor_SMD:C_0603_1608Metric
