File: knobber/MCU.kicad_sch (KiCad schematic)
At the start: 3 parts, among them J801 Conn_01x04_Socket, U801 BMD-340-A-R

Commit message: updated schematic
Parts:
- added C801, C802: 4.7uF, Capacitor_SMD:C_0603_1608Metric, symbol Device:C
- added C804: 0.1uF, Capacitor_SMD:C_0603_1608Metric, symbol Device:C
- added C805: 2.2uF, Capacitor_SMD:C_1206_3216Metric, symbol Device:C
- added J802: Micro_SD_Card, Connector_Card:microSD_HC_Wuerth_693072010801, symbol Connector:Micro_SD_Card
- added R801, R802: 27, Resistor_SMD:R_0402_1005Metric, symbol Device:R
- added R803: 1M, Resistor_SMD:R_1206_3216Metric, symbol Device:R
- added R804, R805, R806, R807: 100k, Resistor_SMD:R_0402_1005Metric, symbol Device:R
- added U802: ESD224DQA, Package_DFN_QFN:Diodes_UDFN-10_1x2.5mm_P0.5mm, symbol Power_Protection:ESD224DQA
- C803: renamed from C801; value 4.7uF -> 10uF; footprint Capacitor_SMD:C_0805_2012Metric -> Capacitor_SMD:C_0603_1608Metric
- J801: footprint (none) -> Connector_PinSocket_2.54mm:PinSocket_1x04_P2.54mm_Vertical
Connections:
- net 3.3V: now also C801.1, C802.1, C804.1, J802.4 (VDD), R804.2, R805.2, R806.2, R807.2
- net GND: now also C801.2, C802.2, C804.2, C805.2, J802.6 (VSS), R803.2, U802.3 (VSS), U802.8 (VSS)
- net USB_D+: now also R801.1; no longer U801.68 (USB-D+)
- net USB_D-: now also R802.1; no longer U801.67 (USB-D-)
- net ~{RESET}: now reaches J801.3 (Pin_3), U801.39 (P0.18)
- net SW_CLK: now reaches U801.43 (SWCLK)
- net SW_CLK: now also J801.2 (Pin_2); no longer J801.1 (Pin_1)
- net SW_DIO: now reaches U801.44 (SWDIO)
- net SW_DIO: now also J801.1 (Pin_1); no longer J801.2 (Pin_2)
- new net: R801.2, U801.68 (USB-D+)
- new net: J802.2 (DAT3/CD), U802.10
- new net: J802.7 (DAT0), U802.6
- new net: J802.5 (CLK), U802.7
- new net: J802.3 (CMD), U802.9
- new net: C805.1, J802.9 (SHIELD), R803.1
- new net: R802.2, U801.67 (USB-D-)
- new net SD_CLK: R805.1, U802.4
- new net SD_MISO: R806.1, U802.5
- new net SD_MOSI: R804.1, U802.2
- new net SD_~{CS}: R807.1, U802.1
- no-connect marks 0 -> 2
Other:
- moved on the sheet: C803
