File: knobber/Motor_driver.kicad_sch (KiCad schematic)
At the start: 17 parts, among them U104 TMC6300-LA-T, U105 LMV321

Commit message: updated schematic
Parts:
- C602: renamed from C604; footprint Capacitor_SMD:C_0805_2012Metric -> Capacitor_SMD:C_0603_1608Metric
- C603: renamed from C602; footprint Capacitor_SMD:C_0805_2012Metric -> Capacitor_SMD:C_0603_1608Metric
- C604: renamed from C603; footprint Capacitor_SMD:C_0805_2012Metric -> Capacitor_SMD:C_0603_1608Metric
- C605: renamed from C105; footprint Capacitor_SMD:C_0805_2012Metric -> Capacitor_SMD:C_0603_1608Metric
- C606: renamed from C601; footprint (none) -> Capacitor_SMD:C_0603_1608Metric
- R601: renamed from R603; footprint Resistor_SMD:R_0603_1608Metric -> Resistor_SMD:R_0402_1005Metric
- R602: renamed from R604; footprint Resistor_SMD:R_0603_1608Metric -> Resistor_SMD:R_0402_1005Metric
- R603: renamed from R605; footprint Resistor_SMD:R_0603_1608Metric -> Resistor_SMD:R_0402_1005Metric
- R604: renamed from R606; footprint Resistor_SMD:R_0603_1608Metric -> Resistor_SMD:R_0402_1005Metric
- R605: renamed from R607; footprint Resistor_SMD:R_0603_1608Metric -> Resistor_SMD:R_0402_1005Metric
- R606: renamed from R608; footprint Resistor_SMD:R_0603_1608Metric -> Resistor_SMD:R_0402_1005Metric
- R607: renamed from R105; footprint Resistor_SMD:R_0603_1608Metric -> Resistor_SMD:R_1206_3216Metric
- U601: renamed from U104; footprint TMC6300-LA-T:QFN40P300X300X90-21N -> TMC6300:QFN40P300X300X90-21N
- renumbered C605 to C601, R601 to R608, R602 to R609, U105 to U602
Connections:
- net Motor_Diag renamed MOT_DIAG
- net Motor_Sens renamed MOT_SENS
- net Motor_U renamed MOT_U
- net Motor_UH renamed MOT_UH
- net Motor_UL renamed MOT_UL
- net Motor_V renamed MOT_V
- net Motor_VH renamed MOT_VH
- net Motor_VL renamed MOT_VL
- net Motor_W renamed MOT_W
- net Motor_WH renamed MOT_WH
- net Motor_WL renamed MOT_WL
Other:
- moved on the sheet: C603
