File: knobber/Power.kicad_sch (KiCad schematic)
At the start: 3 parts, among them U101 AP2112K-3.3

Commit message: updated schematic
Parts:
- renumbered C101 to C501, C102 to C502, U101 to U501
Changed lines of the file:
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@@
+	(wire
+		(pts
+			(xy 91.44 63.5) (xy 91.44 64.77)
+		)
+		(stroke
+			(width 0)
+			(type default)
+		)
+	)
 	(wire
 		(pts
@@
 	(wire
 		(pts
-			(xy 91.44 63.5) (xy 91.44 64.77)
-		)
-		(stroke
-			(width 0)
-			(type default)
-		)
-	)
-	(wire
-		(pts
 			(xy 101.6 67.31) (xy 96.52 67.31)
 		)
@@
 	(wire
 		(pts
-			(xy 88.9 64.77) (xy 91.44 64.77)
-		)
-		(stroke
-			(width 0)
-			(type default)
-		)
-	)
-	(wire
-		(pts
-			(xy 120.65 64.77) (xy 124.46 64.77)
-		)
-		(stroke
-			(width 0)
-			(type default)
-		)
-	)
-	(wire
-		(pts
 			(xy 120.65 74.93) (xy 120.65 77.47)
 		)
@@
 			(width 0)
 			(type default)
-		)
-	)
-	(hierarchical_label "3.3V"
-		(shape output)
-		(at 124.46 64.77 0)
-		(effects
-			(font
-				(size 1.27 1.27)
-			)
-			(justify left)
-		)
-	)
-	(hierarchical_label "5V"
-		(shape input)
-		(at 88.9 64.77 180)
-		(effects
-			(font
-				(size 1.27 1.27)
-			)
-			(justify right)
 		)
 	)
@@
 		(dnp no)
 		(fields_autoplaced yes)
-		(property "Reference" "#PWR0108"
+		(property "Reference" "#PWR0504"
 			(at 120.65 67.31 0)
 			(effects
@@
 			(project "knobber"
 				(path "/09c102b8-dfc1-4666-b1e2-d0c53b401993/85d824be-943a-4d66-829a-99636d7bcd2c"
-					(reference "#PWR0108")
+					(reference "#PWR0504")
 					(unit 1)
 				)
@@
 		(on_board yes)
 		(dnp no)
-		(property "Reference" "C101"
+		(property "Reference" "C501"
 			(at 95.25 69.8499 0)
 			(effects
@@
 			(project "knobber"
 				(path "/09c102b8-dfc1-4666-b1e2-d0c53b401993/85d824be-943a-4d66-829a-99636d7bcd2c"
-					(reference "C101")
+					(reference "C501")
 					(unit 1)
 				)
@@
 		(dnp no)
 		(fields_autoplaced yes)
-		(property "Reference" "#PWR0105"
+		(property "Reference" "#PWR0501"
 			(at 91.44 67.31 0)
 			(effects
@@
 			(project "knobber"
 				(path "/09c102b8-dfc1-4666-b1e2-d0c53b401993/85d824be-943a-4d66-829a-99636d7bcd2c"
-					(reference "#PWR0105")
+					(reference "#PWR0501")
 					(unit 1)
 				)
@@
 		(dnp no)
 		(fields_autoplaced yes)
-		(property "Reference" "#PWR0109"
+		(property "Reference" "#PWR0505"
 			(at 120.65 83.82 0)
 			(effects
@@
 			(project "knobber"
 				(path "/09c102b8-dfc1-4666-b1e2-d0c53b401993/85d824be-943a-4d66-829a-99636d7bcd2c"
-					(reference "#PWR0109")
+					(reference "#PWR0505")
 					(unit 1)
 				)
@@
 		(dnp no)
 		(fields_autoplaced yes)
-		(property "Reference" "#PWR0107"
+		(property "Reference" "#PWR0503"
 			(at 109.22 83.82 0)
 			(effects
@@
 			(project "knobber"
 				(path "/09c102b8-dfc1-4666-b1e2-d0c53b401993/85d824be-943a-4d66-829a-99636d7bcd2c"
-					(reference "#PWR0107")
+					(reference "#PWR0503")
 					(unit 1)
 				)
@@
 		(dnp no)
 		(fields_autoplaced yes)
-		(property "Reference" "U101"
+		(property "Reference" "U501"
 			(at 109.22 58.42 0)
 			(effects
@@
 			(project "knobber"
 				(path "/09c102b8-dfc1-4666-b1e2-d0c53b401993/85d824be-943a-4d66-829a-99636d7bcd2c"
-					(reference "U101")
+					(reference "U501")
 					(unit 1)
 				)
@@
 		(dnp no)
 		(fields_autoplaced yes)
-		(property "Reference" "#PWR0106"
+		(property "Reference" "#PWR0502"
 			(at 91.44 83.82 0)
 			(effects
@@
 			(project "knobber"
 				(path "/09c102b8-dfc1-4666-b1e2-d0c53b401993/85d824be-943a-4d66-829a-99636d7bcd2c"
-					(reference "#PWR0106")
+					(reference "#PWR0502")
 					(unit 1)
 				)
@@
 		(on_board yes)
 		(dnp no)
-		(property "Reference" "C102"
+		(property "Reference" "C502"
 			(at 124.46 69.8499 0)
 			(effects
@@
 			(project "knobber"
 				(path "/09c102b8-dfc1-4666-b1e2-d0c53b401993/85d824be-943a-4d66-829a-99636d7bcd2c"
-					(reference "C102")
-					(unit 1)
-				)
+					(reference "C502")
+					(unit 1)
+				)
