File: knobber/Sensors.kicad_sch (KiCad schematic)
At the start: 6 parts, among them U102 MT6701CT, U103 VEML7700-TT

Commit message: updated schematic
Parts:
- C401: renamed from C103; footprint Capacitor_SMD:C_0805_2012Metric -> Capacitor_SMD:C_0603_1608Metric
- C402: renamed from C104; footprint Capacitor_SMD:C_0805_2012Metric -> Capacitor_SMD:C_0603_1608Metric
- renumbered R103 to R401, R104 to R402, U102 to U401, U103 to U402
