File: knobber/USB.kicad_sch (KiCad schematic)
At the start: 4 parts, among them J101 USB_C_Receptacle_USB2.0_16P

Commit message: updated schematic
Parts:
- removed D101: SP0502BAHT, Package_TO_SOT_SMD:SOT-23, symbol Power_Protection:SP0502BAHT
- added C301: 100nF, Capacitor_SMD:C_0805_2012Metric, symbol Device:C
- added D301: PRTR5V0U2X, Package_TO_SOT_SMD:SOT-143, symbol Power_Protection:PRTR5V0U2X
- R301: renamed from R101; footprint Resistor_SMD:R_0603_1608Metric -> Resistor_SMD:R_0402_1005Metric
- R302: renamed from R102; footprint Resistor_SMD:R_0603_1608Metric -> Resistor_SMD:R_0402_1005Metric
- renumbered J101 to J301
Connections:
- net 5V: now also C301.1, D301.4 (VCC)
- net GND: now also C301.2, D301.1 (GND)
- net USB_D+: now also D301.3 (I/O2)
- net USB_D-: now also D301.2 (I/O1)
Other:
- moved on the sheet: J301, R301, R302
