File: knobber/knobber.kicad_pcb (KiCad board)
At the start: 4 copper layers, 170 x 110 mm, 189 parts, among them J101 BLDC, J301 USB_C_Receptacle_USB2.0_16P, J801 SWD, J802 Micro_SD_Card, J901 LCD, U201 SN74LV1T34DBV, U401 MT6701CT, U402 VEML7700-TT, U501 AP2112K-3.3, U601 TMC6300-LA-T, U602 LMV321, U701 SN74LV1T34DBV, U801 BMD-340-A-R, U802 ESD224DQA

Commit message: Updated schematic and PCB
Parts:
- removed C701, C702, C703, C704, C705, C706, C707, C708, C709, C710, C711, C712, C713, C714, C715, C716, C717, C718, C719, C720, C721: 0.1uF, Capacitor_SMD:C_0603_1608Metric
- removed D701, D702, D703, D704, D705, D706, D707, D708, D709, D710, D711, D712, D713, D714, D715, D716, D717, D718, D719, D720: 1N4148W, Diode_SMD:D_SOD-123
- removed J901: LCD, Connector_PinSocket_2.54mm:PinSocket_1x08_P2.54mm_Vertical
- removed LED701, LED702, LED703, LED704, LED705, LED706, LED707, LED708, LED709, LED710, LED711, LED712, LED713, LED714, LED715, LED716, LED717, LED718, LED719, LED720: choc_SK6812MINI-E, PCM_marbastlib-choc:LED_choc_6028R
- removed MX701, MX702, MX703, MX704, MX705, MX706, MX707, MX708, MX709, MX710, MX711, MX712, MX713, MX714, MX715, MX716, MX717, MX718, MX719, MX720: MX_SW_HS, PCM_marbastlib-mx:SW_MX_HS_CPG151101S11_1u
- removed TP601: MOT_UH, TestPoint:TestPoint_Pad_D1.0mm
- removed TP602: MOT_UL, TestPoint:TestPoint_Pad_D1.0mm
- removed TP603: MOT_VH, TestPoint:TestPoint_Pad_D1.0mm
- removed TP604: MOT_VL, TestPoint:TestPoint_Pad_D1.0mm
- removed TP605: MOT_WH, TestPoint:TestPoint_Pad_D1.0mm
- removed TP606: MOT_WL, TestPoint:TestPoint_Pad_D1.0mm
- removed TP608: MOT_DIAG, TestPoint:TestPoint_Pad_D1.0mm
- removed TP701: LED_DATA, TestPoint:TestPoint_Pad_D1.0mm
- removed U701: SN74LV1T34DBV, Package_TO_SOT_SMD:SOT-23-5
- C801: value 4.7uF -> 10uF
- C802: value 4.7uF -> 0.1uF
- C803: value 10uF -> 4.7uF
- C804: value 0.1uF -> 4.7uF
- moved D213 358.3 mm to (97.0, 105.3), turned to 90 degrees
- moved D214 353.0 mm to (100.0, 90.0), turned to 67.5 degrees
- moved D212 348.6 mm to (100.0, 120.6), turned to 112.5 degrees
- moved D215 343.4 mm to (108.7, 77.0), turned to 45 degrees
- moved D211 343.1 mm to (108.7, 133.6), turned to 135 degrees
- moved C203 337.9 mm to (93.3, 104.3), turned to -90 degrees
- moved C202 336.7 mm to (96.5, 121.2), turned to -67.5 degrees
- moved C217 336.4 mm to (105.7, 135.3), turned to -45 degrees
- moved D210 333.4 mm to (121.7, 142.3), turned to 157.5 degrees
- moved C204 333.4 mm to (97.1, 87.8), turned to -112.5 degrees
- moved D216 330.3 mm to (121.7, 68.3), turned to 22.5 degrees
- moved C216 324.7 mm to (119.6, 145.0), turned to -22.5 degrees
- moved C205 323.8 mm to (106.9, 73.8), turned to -135 degrees
- moved D209 320.7 mm to (137.0, 145.3), turned to 180 degrees
- moved C215 309.9 mm to (136.1, 148.5)
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Connections:
- C804 pad 1: 3.3V -> 5V
- D301 pad 2: /USB/USB_D- -> /MCU/USB_D-
- D301 pad 3: /USB/USB_D+ -> /MCU/USB_D+
- J301 pad A6: /USB/USB_D+ -> /MCU/USB_D+
- J301 pad A7: /USB/USB_D- -> /MCU/USB_D-
- J301 pad B6: /USB/USB_D+ -> /MCU/USB_D+
- J301 pad B7: /USB/USB_D- -> /MCU/USB_D-
- U801 pad 10: unconnected-(U801-P0.29-Pad10) -> /MCU/P0.29
- U801 pad 11: unconnected-(U801-P0.30-Pad11) -> /MCU/P0.30
- U801 pad 12: unconnected-(U801-P0.31-Pad12) -> /MCU/P0.31
- U801 pad 13: unconnected-(U801-P0.00-Pad13) -> /MCU/P0.00
- U801 pad 14: unconnected-(U801-P0.01-Pad14) -> /MCU/P0.01
- U801 pad 15: unconnected-(U801-P0.02-Pad15) -> /MCU/P0.02
- U801 pad 19: unconnected-(U801-P0.03-Pad19) -> /MCU/P0.03
- U801 pad 20: unconnected-(U801-P0.04-Pad20) -> /MCU/P0.04
- U801 pad 21: unconnected-(U801-P0.05-Pad21) -> /MCU/P0.05
- U801 pad 22: unconnected-(U801-P0.06-Pad22) -> /MCU/P0.06
- U801 pad 23: unconnected-(U801-P0.07-Pad23) -> /MCU/P0.07
- U801 pad 24: unconnected-(U801-P0.08-Pad24) -> /MCU/P0.08
- U801 pad 25: unconnected-(U801-P0.09-Pad25) -> /MCU/P0.09
- U801 pad 26: unconnected-(U801-P0.10-Pad26) -> /MCU/P0.10
- U801 pad 27: unconnected-(U801-P0.11-Pad27) -> /MCU/P0.11
- U801 pad 28: unconnected-(U801-P0.12-Pad28) -> /MCU/P0.12
- U801 pad 31: unconnected-(U801-P0.13-Pad31) -> /MCU/P0.13
- U801 pad 32: unconnected-(U801-P0.14-Pad32) -> /MCU/P0.14
- U801 pad 33: unconnected-(U801-P0.15-Pad33) -> /MCU/P0.15
- U801 pad 34: unconnected-(U801-P0.16-Pad34) -> /MCU/P0.16
- U801 pad 35: unconnected-(U801-P0.17-Pad35) -> /MCU/P0.17
- U801 pad 36: unconnected-(U801-P0.21-Pad36) -> /MCU/P0.21
- U801 pad 37: unconnected-(U801-P0.19-Pad37) -> /MCU/P0.19
- U801 pad 38: unconnected-(U801-P0.20-Pad38) -> /MCU/P0.20
- U801 pad 40: unconnected-(U801-P0.22-Pad40) -> /MCU/P0.22
- U801 pad 41: unconnected-(U801-P0.23-Pad41) -> /MCU/P0.23
- U801 pad 42: unconnected-(U801-P0.24-Pad42) -> /MCU/P0.24
- U801 pad 48: unconnected-(U801-P1.05-Pad48) -> /MCU/P1.05
- U801 pad 49: unconnected-(U801-P1.06-Pad49) -> /MCU/P1.06
- U801 pad 50: unconnected-(U801-P1.07-Pad50) -> /MCU/P1.07
- U801 pad 51: unconnected-(U801-P1.08-Pad51) -> /MCU/P1.08
- U801 pad 52: unconnected-(U801-P1.09-Pad52) -> /MCU/P1.09
- U801 pad 53: unconnected-(U801-P1.10-Pad53) -> /MCU/P1.10
- U801 pad 54: unconnected-(U801-P1.11-Pad54) -> /MCU/P1.11
- U801 pad 56: unconnected-(U801-P1.00-Pad56) -> /MCU/P1.00
- U801 pad 57: unconnected-(U801-P1.01-Pad57) -> /MCU/P1.01
- U801 pad 58: unconnected-(U801-P1.02-Pad58) -> /MCU/P1.02
- U801 pad 59: unconnected-(U801-P1.03-Pad59) -> /MCU/P1.03
- U801 pad 6: unconnected-(U801-P0.25-Pad6) -> /MCU/P0.25
- U801 pad 60: unconnected-(U801-P1.04-Pad60) -> /MCU/P1.04
- U801 pad 61: unconnected-(U801-P1.12-Pad61) -> /MCU/P1.12
- U801 pad 62: unconnected-(U801-P1.13-Pad62) -> /MCU/P1.13
- U801 pad 63: unconnected-(U801-P1.14-Pad63) -> /MCU/P1.14
- U801 pad 64: unconnected-(U801-P1.15-Pad64) -> /MCU/P1.15
- U801 pad 65: 3.3V -> 5V
- U801 pad 7: unconnected-(U801-P0.26-Pad7) -> /MCU/P0.26
- U801 pad 8: unconnected-(U801-P0.27-Pad8) -> /MCU/P0.27
- U801 pad 9: unconnected-(U801-P0.28-Pad9) -> /MCU/P0.28
Routing:
- net /MCU/USB_D+: track 0.00 -> 16.9 mm
- net /USB/USB_D+: track 16.9 -> 0.00 mm
- net /USB/USB_D-: track 16.6 -> 0.00 mm
- net /MCU/USB_D-: track 0.00 -> 16.6 mm
- net unconnected-(U801-P0.03-Pad19): track 6.49 -> 0.00 mm
- net /MCU/P0.03: track 0.00 -> 6.49 mm
- net unconnected-(U801-P0.05-Pad21): track 6.35 -> 0.00 mm
- net /MCU/P0.05: track 0.00 -> 6.35 mm
- net unconnected-(U801-P0.07-Pad23): track 6.29 -> 0.00 mm
- net /MCU/P0.07: track 0.00 -> 6.29 mm
- net unconnected-(U801-P0.09-Pad25): track 6.23 -> 0.00 mm
- net /MCU/P0.09: track 0.00 -> 6.23 mm
- net unconnected-(U801-P0.01-Pad14): track 5.90 -> 0.00 mm
- net /MCU/P0.01: track 0.00 -> 5.90 mm
- net unconnected-(U801-P0.31-Pad12): track 5.80 -> 0.00 mm
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